Commit message: Include Isaac-Sim

File: jaka_lumi_ros/src/jaka_lumi_description/urdf/jaka_lumi.urdf (robot description, URDF)
Before this commit: robot jaka_lumi, 14 links, 13 joints
Links:
- removed link link-1
- removed link link-2
- removed link link-3
- removed link link-4
- removed link link-a1
- removed link link-a2
- removed link link-a3
- removed link link-a4
- removed link link-a5
- removed link link-a6
- removed link link-at
- removed link wheel-l
- removed link wheel-r
- added link link_1, mass 14.2347501496821; collision mesh filename=package://jaka_lumi_description/meshes/link_1.STL; visual mesh filename=package://jaka_lumi_description/meshes/link_1.STL
- added link link_2, mass 4.81096378907801; collision mesh filename=package://jaka_lumi_description/meshes/link_2.STL; visual mesh filename=package://jaka_lumi_description/meshes/link_2.STL
- added link link_3, mass 1.2679984054123; collision mesh filename=package://jaka_lumi_description/meshes/link_3.STL; visual mesh filename=package://jaka_lumi_description/meshes/link_3.STL
- added link link_4, mass 0.595955123537826; collision mesh filename=package://jaka_lumi_description/meshes/link_4.STL; visual mesh filename=package://jaka_lumi_description/meshes/link_4.STL
- added link link_a1, mass 1.35363412771609; collision mesh filename=package://jaka_lumi_description/meshes/link_a1.STL; visual mesh filename=package://jaka_lumi_description/meshes/link_a1.STL
- added link link_a2, mass 1.13725613291731; collision mesh filename=package://jaka_lumi_description/meshes/link_a2.STL; visual mesh filename=package://jaka_lumi_description/meshes/link_a2.STL
- added link link_a3, mass 0.81274798684902; collision mesh filename=package://jaka_lumi_description/meshes/link_a3.STL; visual mesh filename=package://jaka_lumi_description/meshes/link_a3.STL
- added link link_a4, mass 0.308941204464269; collision mesh filename=package://jaka_lumi_description/meshes/link_a4.STL; visual mesh filename=package://jaka_lumi_description/meshes/link_a4.STL
- added link link_a5, mass 0.691485853906912; collision mesh filename=package://jaka_lumi_description/meshes/link_a5.STL; visual mesh filename=package://jaka_lumi_description/meshes/link_a5.STL
- added link link_a6, mass 0.147762214293587; collision mesh filename=package://jaka_lumi_description/meshes/link_a6.STL; visual mesh filename=package://jaka_lumi_description/meshes/link_a6.STL
- added link link_at, mass 0.00155862265526224; collision mesh filename=package://jaka_lumi_description/meshes/link_at.STL; visual mesh filename=package://jaka_lumi_description/meshes/link_at.STL
- added link wheel_l, mass 0.941042738950082; collision mesh filename=package://jaka_lumi_description/meshes/wheel_l.STL; visual mesh filename=package://jaka_lumi_description/meshes/wheel_l.STL
- added link wheel_r, mass 0.941042738950082; collision mesh filename=package://jaka_lumi_description/meshes/wheel_r.STL; visual mesh filename=package://jaka_lumi_description/meshes/wheel_r.STL
- added link world
Joints:
- removed joint l-1
- removed joint l-2
- removed joint l-3
- removed joint l-4
- removed joint l-a1
- removed joint l-a2
- removed joint l-a3
- removed joint l-a4
- removed joint l-a5
- removed joint l-a6
- removed joint l-at
- removed joint w-l
- removed joint w-r
- added joint fixed: type fixed, parent world, child base_link
- added joint l_1: type prismatic, parent base_link, child link_1, origin xyz=0 0 0.565 rpy=0 0 0, axis 0 0 1, limit lower=0 upper=0.4 effort=0 velocity=0
- added joint l_2: type revolute, parent link_1, child link_2, origin xyz=0 0 0.0745 rpy=0 0 0, axis 0 0 1, limit lower=-2.7925 upper=2.7925 effort=0 velocity=0
- added joint l_3: type revolute, parent link_2, child link_3, origin xyz=0 0 0.3465 rpy=0 0 0, axis 0 0 1, limit lower=-3.1415 upper=3.1415 effort=0 velocity=0
- added joint l_4: type revolute, parent link_3, child link_4, origin xyz=0 0 0.052 rpy=0 1.5708 0, axis 0 0 1, limit lower=-0.0872 upper=0.6108 effort=0 velocity=0
- added joint l_a1: type revolute, parent link_2, child link_a1, origin xyz=-0.104 0 0.069 rpy=3.1416 1.5708 0, axis 0 0 1, limit lower=-6.2831 upper=6.2831 effort=0 velocity=0
- added joint l_a2: type revolute, parent link_a1, child link_a2, origin xyz=0 -0.0165 0.156 rpy=1.5708 -1.5708 0, axis 0 0 1, limit lower=-2.1816 upper=2.1816 effort=0 velocity=0
- added joint l_a3: type revolute, parent link_a2, child link_a3, origin xyz=0.21 0 -0.029 rpy=0 0 0, axis 0 0 1, limit lower=-2.2689 upper=2.2689 effort=0 velocity=0
- added joint l_a4: type revolute, parent link_a3, child link_a4, origin xyz=0.1303 0 0.0185 rpy=-1.5708 0 -1.5708, axis 0 0 1, limit lower=-6.2831 upper=6.2831 effort=0 velocity=0
- added joint l_a5: type revolute, parent link_a4, child link_a5, origin xyz=0 -0.01805 0.0802 rpy=1.5708 1.5708 0, axis 0 0 1, limit lower=-2.0943 upper=2.0943 effort=0 velocity=0
- added joint l_a6: type revolute, parent link_a5, child link_a6, origin xyz=-0.1233 0 0.01805 rpy=1.5708 0 -1.5708, axis 0 0 1, limit lower=-6.2831 upper=6.2831 effort=0 velocity=0
- added joint l_at: type fixed, parent link_a6, child link_at, origin xyz=0 0 0.036 rpy=0 0 0, axis 0 0 0
- added joint w_l: type continuous, parent base_link, child wheel_l, origin xyz=0.1793 0.050006 -0.2071 rpy=0 1.5708 0, axis 0 0 1
- added joint w_r: type continuous, parent base_link, child wheel_r, origin xyz=-0.1793 0.050006 -0.2071 rpy=0 1.5708 0, axis 0 0 1

File: jaka_lumi_ros/src/jaka_lumi_moveit_config/config/jaka_lumi.ros2_control.xacro (robot description, xacro)
@@ -1,5 +1,5 @@
 <?xml version="1.0"?>
 <robot xmlns:xacro="http://www.ros.org/wiki/xacro">
-    <xacro:macro name="jaka_lumi_ros2_control" params="name initial_positions_file use_gazebo use_rviz_sim">
+    <xacro:macro name="jaka_lumi_ros2_control" params="name initial_positions_file use_gazebo use_rviz_sim use_isaac_sim">
         <xacro:property name="initial_positions" value="${xacro.load_yaml(initial_positions_file)['initial_positions']}"/>
         <ros2_control name="${name}" type="system">
@@ -8,79 +8,98 @@
               <xacro:if value="${use_gazebo}">
                   <!-- <plugin>gazebo_ros2_control/GazeboSystem</plugin> -->
-                  <!-- <plugin>ign_ros2_control/IgnitionSystem</plugin> -->
-                  <plugin>gz_ros2_control/GazeboSimSystem</plugin>
+                  <plugin>ign_ros2_control/IgnitionSystem</plugin>
+                  <!-- <plugin>gz_ros2_control/GazeboSimSystem</plugin> -->
               </xacro:if>
               <xacro:if value="${use_rviz_sim}">
                   <plugin>mock_components/GenericSystem</plugin>
               </xacro:if>
+              <xacro:if value="${use_isaac_sim}">
+                <plugin>topic_based_ros2_control/TopicBasedSystem</plugin>
+                <param name="joint_states_topic">/isaac_joint_states</param>
+                <param name="joint_commands_topic">/isaac_joint_commands</param>
+              </xacro:if>
             </hardware>
             <!-- Joint interfaces generated for each joint -->
-            <joint name="l-1">
+            <!-- <joint name="w_r">
                 <command_interface name="position"/>
                 <state_interface name="position">
-                  <param name="initial_value">${initial_positions['l-1']}</param>
+                  <param name="initial_value">${initial_positions['w_r']}</param>
                 </state_interface>
                 <state_interface name="velocity"/>
             </joint>
-            <joint name="l-2">
+            <joint name="w_l">
                 <command_interface name="position"/>
                 <state_interface name="position">
-                  <param name="initial_value">${initial_positions['l-2']}</param>
+                  <param name="initial_value">${initial_positions['w_l']}</param>
+                </state_interface>
+                <state_interface name="velocity"/>
+            </joint> -->
+            <joint name="l_1">
+                <command_interface name="position"/>
+                <state_interface name="position">
+                  <param name="initial_value">${initial_positions['l_1']}</param>
                 </state_interface>
                 <state_interface name="velocity"/>
             </joint>
-            <joint name="l-3">
+            <joint name="l_2">
                 <command_interface name="position"/>
                 <state_interface name="position">
-                  <param name="initial_value">${initial_positions['l-3']}</param>
+                  <param name="initial_value">${initial_positions['l_2']}</param>
                 </state_interface>
                 <state_interface name="velocity"/>
             </joint>
-            <joint name="l-4">
+            <joint name="l_3">
                 <command_interface name="position"/>
                 <state_interface name="position">
-                  <param name="initial_value">${initial_positions['l-4']}</param>
+                  <param name="initial_value">${initial_positions['l_3']}</param>
                 </state_interface>
                 <state_interface name="velocity"/>
             </joint>
-            <joint name="l-a1">
+            <joint name="l_4">
                 <command_interface name="position"/>
                 <state_interface name="position">
-                  <param name="initial_value">${initial_positions['l-a1']}</param>
+                  <param name="initial_value">${initial_positions['l_4']}</param>
                 </state_interface>
                 <state_interface name="velocity"/>
             </joint>
-            <joint name="l-a2">
+            <joint name="l_a1">
                 <command_interface name="position"/>
                 <state_interface name="position">
-                  <param name="initial_value">${initial_positions['l-a2']}</param>
+                  <param name="initial_value">${initial_positions['l_a1']}</param>
                 </state_interface>
                 <state_interface name="velocity"/>
             </joint>
-            <joint name="l-a3">
+            <joint name="l_a2">
                 <command_interface name="position"/>
                 <state_interface name="position">
-                  <param name="initial_value">${initial_positions['l-a3']}</param>
+                  <param name="initial_value">${initial_positions['l_a2']}</param>
                 </state_interface>
                 <state_interface name="velocity"/>
             </joint>
-            <joint name="l-a4">
+            <joint name="l_a3">
                 <command_interface name="position"/>
                 <state_interface name="position">
-                  <param name="initial_value">${initial_positions['l-a4']}</param>
+                  <param name="initial_value">${initial_positions['l_a3']}</param>
                 </state_interface>
                 <state_interface name="velocity"/>
             </joint>
-            <joint name="l-a5">
+            <joint name="l_a4">
                 <command_interface name="position"/>
                 <state_interface name="position">
-                  <param name="initial_value">${initial_positions['l-a5']}</param>
+                  <param name="initial_value">${initial_positions['l_a4']}</param>
                 </state_interface>
                 <state_interface name="velocity"/>
             </joint>
-            <joint name="l-a6">
+            <joint name="l_a5">
                 <command_interface name="position"/>
                 <state_interface name="position">
-                  <param name="initial_value">${initial_positions['l-a6']}</param>
+                  <param name="initial_value">${initial_positions['l_a5']}</param>
+                </state_interface>
+                <state_interface name="velocity"/>
+            </joint>
+            <joint name="l_a6">
+                <command_interface name="position"/>
+                <state_interface name="position">
+                  <param name="initial_value">${initial_positions['l_a6']}</param>
                 </state_interface>
                 <state_interface name="velocity"/>

File: jaka_lumi_ros/src/jaka_lumi_moveit_config/config/jaka_lumi.urdf.xacro (robot description, xacro)
@@ -4,4 +4,5 @@
     <xacro:arg name="use_gazebo" default="false"/>
     <xacro:arg name="use_rviz_sim" default="false"/>
+    <xacro:arg name="use_isaac_sim" default="false"/>
     <!-- Import jaka_lumi urdf file -->
     <xacro:include filename="$(find jaka_lumi_description)/urdf/jaka_lumi.urdf" />
@@ -9,4 +10,4 @@
     <xacro:include filename="jaka_lumi.ros2_control.xacro" />
     <!-- <xacro:jaka_lumi_ros2_control name="FakeSystem" initial_positions_file="$(arg initial_positions_file)"/> -->
-    <xacro:jaka_lumi_ros2_control name="jaka_lumi_hardware" initial_positions_file="$(arg initial_positions_file)" use_gazebo="$(arg use_gazebo)" use_rviz_sim="$(arg use_rviz_sim)" />
+    <xacro:jaka_lumi_ros2_control name="jaka_lumi_hardware" initial_positions_file="$(arg initial_positions_file)" use_gazebo="$(arg use_gazebo)" use_rviz_sim="$(arg use_rviz_sim)" use_isaac_sim="$(arg use_isaac_sim)" />
 </robot>
